File: hardware/sv16_board/sv16_board.kicad_sch (KiCad schematic)
At the start: 132 parts, among them J1 JTAG, J10 CONSOLE, J2 JTAG-1.27, J3 EXP-A, J4 EXP-B, J5 EXP-C, J6 MOTOR, J8 USB-C, J9 7-12 V, Q1 2N7002, Q2 BC817, Q4 BC807, SW1 RESET, SW2 RECONFIG, U1 LFE5U-12F-6TG144C, U2 W25Q64JVSSIQ, U3 W25Q64JVSSIQ, U4 CH340G, U5 AP62300TWU-7, U6 MP1584EN, U7 LP5907MFX-2.5, U8 USBLC6-2SC6, Y1 25 MHz ACTIVE XO (4-pin), Y2 12 MHz (CH340G clock)

Commit message: WIP: draw real wires between pins in the KiCad schematic
Wave 11.  The schematic now joins pins with drawn wire segments instead
of dropping a global label on every pin.

Adds an orthogonal grid router that may cross another net at right
angles but never runs along it (which would silently merge two nets),
a keep-out margin around every symbol body, and a short reserved exit
corridor per pin so a pin can never be sealed in by other wiring.
Junctions are placed automatically wherever three or more wire ends
meet.

175 of the 256 signal pins are now drawn wires; 33 of 118 nets still
fall back to labels because the router cannot find a path for them.
The 216 supply pins use rail symbols, which is normal practice.

Co-authored-by: arena-agent <297053741+arena-agent@users.noreply.github.com>
Parts:
- added FID1, FID2, FID3, FID4: (no value), Fiducial:Fiducial_1mm_Mask2mm, symbol SV16:S1
- added H1, H2, H3, H4: (no value), MountingHole:MountingHole_3.2mm_M3, symbol SV16:S1
- added J7: SPARE (not fitted), Connector_PinHeader_2.54mm:PinHeader_2x25_P2.54mm_Vertical, symbol SV16:S8
- added R20, R35: (no value), Resistor_SMD:R_0603_1608Metric, symbol SV16:S0
- C1, C10, C11, C12, C13, C14, C15, C16, C17, C18, C19, C2, C20, C21, C22, C23, C24, C25, C26, C27, C28, C29, C3, C30, C31, C32, C33, C34, C35, C36, C37, C38, C39, C4, C40, C41, C42, C5, C6, C7, C8, C9, D1, D11, D2, D3, D4, D5, D6, D7, D8, D9, FB1, JP1, L1, L2, R1, R10, R11, R12, R13, R14, R15, R16, R17, R18, R19, R2, R21, R22, R23, R24, R25, R26, R27, R28, R29, R3, R30, R31, R32, R33, R34, R36, R37, R38, R39, R4, R40, R41, R43, R44, R45, R46, R47, R48, R49, R5, R6, R7, R8, R9, Y2: symbol SV16:P2_2 -> SV16:S0
- J1: symbol SV16:P10_10 -> SV16:S2
- J10, SW1, SW2, Y1: symbol SV16:P4_1 -> SV16:S11
- J2: symbol SV16:P10_10 -> SV16:S3
- J3: symbol SV16:P20_11 -> SV16:S4
- J4: symbol SV16:P20_11 -> SV16:S5
- J5: symbol SV16:P10_10 -> SV16:S6
- J6: symbol SV16:P6_4 -> SV16:S7
- J8: symbol SV16:P20_7 -> SV16:S9
- J9, Q1, Q2, Q4: symbol SV16:P3_3 -> SV16:S10
- TP1, TP2, TP3, TP4, TP5, TP6: symbol SV16:P1_12 -> SV16:S1
- U1: symbol SV16:P144_0 -> SV16:S12
- U2: symbol SV16:P8_9 -> SV16:S13
- U3: symbol SV16:P8_9 -> SV16:S14
- U4: symbol SV16:P16_8 -> SV16:S15
- U5, U8: symbol SV16:P6_4 -> SV16:S16
- U6: symbol SV16:P9_5 -> SV16:S17
- U7: symbol SV16:P5_6 -> SV16:S18
Connections:
- net D6_K is gone; now on net Q4_C: D6.1, R34.1
- net Q1_G is gone; now on net J10_TX: Q1.2, R25.2, R26.1
- net Q2_B is gone; now on an unnamed net: Q2.2, R32.2
- net Q4_B is gone; now on net Q4_C: Q4.2, R31.2
- net led[0]_k is gone; now on net led[0]: D2.1, R27.2
- net led[1]_k is gone; now on net led[1]: D3.1, R28.2
- net led[2]_k is gone; now on net led[2]: D4.1, R29.2
- net A2: now also R12.1, R13.2, R14.1, R14.2, R15.1, U2.7, U2.8; no longer J5.3, U1.26
- net CC1: no longer J8.A12
- net CCLK: no longer U1.19
- net CFG_0: no longer U1.11
- net CFG_1: no longer U1.14
- net CFG_2: no longer U1.15
- net J10_TX: now also J10.3, J8.S3, J8.S4, Q1.1, R22.2, R23.2, R24.1, R26.2; no longer J10.1
- net Q4_C: now also Q4.1, R34.2; no longer Q4.3
- net TCK: no longer J1.8, J2.1, U1.10
- net TDI: no longer J1.3, J2.3, U1.12
- net TDO: no longer J1.4, J2.2, U1.13
- net TMS: no longer J1.10, J2.4, U1.9
- net U3_HOLD: no longer U3.6
- net U3_WP: no longer U3.2
- net U4_DTR: no longer U4.12
- net U4_RXD: no longer U4.6
- net U4_V3: no longer U4.5
- net U6_EN: no longer U6.4
- net U6_FREQ: no longer U6.9
- net USB_DP_F: now also U8.6; no longer U4.4, U8.4
- net clk_25m: now also Y1.3; no longer U1.84, Y1.4
- net ext_rst_n: no longer SW1.2, U1.83
- net flash_cs_n: no longer U1.106, U3.4
- net led[0]: now also D2.2; no longer U1.34
- net led[1]: now also D3.2; no longer U1.33
- net led[2]: now also D4.2; no longer U1.32
- net led[3]: no longer U1.29
- net motor_fault_n: no longer J6.4, U1.114
- net uart_rx: no longer U1.144
- net at J2.7: now also J5.9
- net at J2.8: now also J5.10
- net at U1.135: now also J3.5, J4.3, U1.99
- removed net 1V1: C2.1, C21.1, C3.1, C4.1, C5.1, C6.1, C7.1, L2.2, R38.1, TP3.1, U1.134, U1.35, U1.44, U1.53, U1.7, U1.87
- removed net 2V5: C10.1, C11.1, C22.1, C42.1, C8.1, C9.1, TP2.1, U1.121, U1.20, U1.56, U1.85, U7.4
- removed net 3V3: C12.1, C13.1, C14.1, C15.1, C16.1, C17.1, C18.1, C19.1, C20.1, C24.1, C25.1, C26.1, C27.1, C28.1, C29.1, C30.1, C40.1, C41.1, D2.2, D3.2, D4.2, D5.2, J1.5, J10.2, J2.5, J3.10, J4.10, J5.6, L1.2, Q4.1, R1.2, R13.2, R14.2, R15.2, R16.2, R17.2, R18.2, R19.2, R2.2, R3.2, R33.1, R4.2, R43.1, R44.1, R46.1, R5.2, R8.2, TP1.1, U1.117, U1.131, U1.3, U1.30, U1.37, U1.57, U1.64, U1.80, U1.95, U2.5, U3.5, U4.9, U7.3, Y1.2, Y1.3
- removed net 5V_USB: J3.13, J3.14, J4.11
- net A0: no longer names the net of J5.5
- net A0: no longer U1.28
- removed net A1: J5.4, R11.1, U1.27
- net A10: no longer names the net of J3.6
- net A10: no longer U1.118
- net A11: no longer names the net of U1.113
- net A11: no longer J3.5
- net A12: no longer names the net of J3.4
- net A12: no longer U1.112
- net A13: no longer names the net of J3.3
- net A13: no longer U1.111
- net A14: no longer names the net of J3.2
- net A14: no longer U1.110
- net A15: no longer names the net of J3.1
- net A15: no longer U1.109
- net A3: no longer names the net of J5.2
- net A3: no longer U1.25
- removed net A4: J5.1, R12.1, U1.24
- removed net A5: J5.10, U1.23
- removed net A6: J5.9, U1.22
- net A7: no longer names the net of J5.8
- net A7: no longer U1.21
- net A8: no longer names the net of J3.8
- net A8: no longer U1.120
- net A9: no longer names the net of J3.7
- net A9: no longer U1.119
- net B0: no longer names the net of J4.8
- net B0: no longer U1.82
- net B1: no longer names the net of J4.7
- net B1: no longer U1.81
- net B10: no longer names the net of J4.18
- net B10: no longer U1.91
- net B11: no longer names the net of J4.17
- net B11: no longer U1.90
- net B12: no longer names the net of J4.16
- net B12: no longer U1.72
- net B13: no longer names the net of J4.15
- net B13: no longer U1.71
- net B14: no longer names the net of J4.14
- net B14: no longer U1.70
- net B15: no longer names the net of J4.13
- net B15: no longer U1.69
- net B2: no longer names the net of J4.6
- net B2: no longer U1.78
- net B3: no longer names the net of J4.5
- net B3: no longer U1.77
- net B4: no longer names the net of J4.4
- net B4: no longer U1.76
- net B5: no longer names the net of U1.75
- net B5: no longer J4.3
- net B6: no longer names the net of J4.2
- net B6: no longer U1.74
- net B7: no longer names the net of J4.1
- net B7: no longer U1.89
- net B8: no longer names the net of J4.20
- net B8: no longer U1.93
- net B9: no longer names the net of J4.19
- net B9: no longer U1.92
- net CC2: no longer names the net of R37.1
- net CC2: no longer J8.S4
- net D1_A: no longer names the net of D1.2, R33.2
- net D1_A: now also Q2.1, R33.1
- net D7_A: no longer names the net of D7.2, R44.2
- net D7_A: now also R44.1
- removed net DONE: J1.7, R32.1, R4.1, TP5.1, U1.17
- net DTR_F: no longer names the net of R25.1
- net DTR_F: no longer JP1.2
- removed net FB_1V1: R38.2, R39.1, U6.2
- removed net GND: C1.2, C10.2, C11.2, C12.2, C13.2, C14.2, C15.2, C16.2, C17.2, C18.2, C19.2, C2.2, C20.2, C21.2, C22.2, C23.2, C24.2, C25.2, C26.2, C27.2, C28.2, C29.2, C3.2, C30.2, C31.2, C32.2, C34.2, C35.2, C36.2, C37.2, C39.2, C4.2, C40.2, C41.2, C42.2, C5.2, C6.2, C7.2, C8.2, C9.2, D11.2, D7.1, J1.9, J10.3, J2.10, J2.6, J3.11, J3.12, J3.15, J3.16, J3.9, J4.12, J4.9, J5.7, J6.2, J8.A4, J8.A5, J8.B4, J8.B5, J8.B6, J8.B7, J8.B8, J8.B9, J9.1, Q1.1, Q2.1, R26.2, R34.2, R36.2, R37.2, R39.2, R40.2, R45.2, R47.2, R49.2, R6.2, R7.2, SW1.1, SW2.1, TP4.1, U1.116, U1.130, U1.132, U1.142, U1.31, U1.41, U1.52, U1.58, U1.65, U1.79, U1.8, U1.86, U1.88, U1.94, U2.1, U3.1, U4.8, U5.3, U6.1, U6.6, U7.2, U8.2, Y1.1
- removed net INITN: J1.6, R3.1, R31.1, TP6.1, U1.18
- net J10_RX: no longer names the net of J10.4
- net J10_RX: no longer R22.2
- net J9_VIN: no longer names the net of J9.2
- net J9_VIN: no longer D8.2
- removed net PROGRAMN: J1.2, Q1.3, R2.1, SW2.2, U1.16
- net Q2_C: no longer names the net of D1.1
- net Q2_C: no longer Q2.3
- net U2_CLK: no longer names the net of R9.2
- net U2_CLK: no longer U2.7
- removed net U2_CS: R12.2, R13.1, U2.4
- net U2_DI: no longer names the net of R10.2
- net U2_DI: no longer U2.8
- net U2_DO: no longer names the net of U2.3
- net U2_DO: no longer R11.2
- net U2_HOLD: no longer names the net of U2.6
- net U2_HOLD: no longer R15.1
- net U2_WP: no longer names the net of U2.2
- net U2_WP: no longer R14.1
- net U4_TXD: no longer names the net of U4.7
- net U4_TXD: no longer R21.1
- net U5_BST: no longer names the net of C38.1
- net U5_BST: now also L1.2, U5.6; no longer U5.4
- removed net U5_EN: R48.2, R49.1, U5.5
- removed net U5_FB: R46.2, R47.1, U5.6
- removed net U5_SW: C38.2, L1.1, U5.2
- net U6_BST: no longer names the net of U6.7
- net U6_BST: no longer C33.1
- removed net U6_COMP: C35.1, R45.1, U6.3
- removed net U6_SW: C33.2, D11.1, L2.1, U6.5
- removed net U7_EN: C32.1, R43.2, U7.1
- removed net USB_DN: J8.A8, J8.S2, U8.1
- net USB_DN_F: no longer names the net of U4.3
- net USB_DN_F: no longer U8.6
- removed net USB_DP: J8.A9, J8.S3, U8.3
- removed net USB_VBUS: D9.2, J8.A1, J8.A6, J8.B1, J8.B12, U8.5
- removed net VM_IN: C23.1, C39.1, FB1.2, J6.3, R41.1, R48.1, U5.1, U6.8
- removed net VM_IN_RAW: D8.1, D9.1, FB1.1
- removed net Y2_XI: C36.1, U4.2, Y2.1
- removed net Y2_XO: C37.1, U4.1, Y2.2
- net flash_miso: no longer names the net of U3.3
- net flash_miso: now also J6.1; no longer U1.104
- net flash_mosi: no longer names the net of U1.105
- net flash_mosi: no longer U3.8
- net flash_sck: no longer names the net of U1.107
- net flash_sck: no longer U3.7
- net led[3]_k: no longer names the net of D5.1
- net led[3]_k: no longer R30.2
- net motor_dir1: no longer names the net of J6.6
- net motor_dir1: no longer U1.128
- net motor_dir2: no longer names the net of J6.5
- net motor_dir2: no longer U1.115
- net pwm_out: no longer names the net of U1.129
- net pwm_out: no longer J6.1
- net spi0_cs_n: no longer names the net of J3.20
- net spi0_cs_n: no longer U1.102
- net spi0_miso: no longer names the net of J3.17
- net spi0_miso: no longer U1.100
- net spi0_mosi: no longer names the net of J3.18
- net spi0_mosi: no longer U1.101
- net spi0_sck: no longer names the net of J3.19
- net spi0_sck: no longer U1.103
- removed net uart_tx: R23.2, R24.1, U1.143
- new net: J6.2, U3.4
- new net: C33.1, U6.8
Other:
- moved on the sheet: C1, C10, C11, C12, C13, C14, C15, C16, C17, C18, C19, C2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

Commit message: Place parts next to the parts they talk to; draw 224 of 256 signal pins
Four placement bugs were making the sheet unroutable:

- The sign on the peripheral offset was inverted, so every connector sat
  on the opposite side of the FPGA from its own pins and every FPGA net
  had to cross the whole chip.
- Connector bodies were drawn at the FPGA's origin while their pins sat
  far below it, making each rectangle ~300 mm tall and overlapping its
  neighbours.
- The straight-wire fast path never checked that the run was clear, so
  it happily drew through symbol bodies (J10_RX ran through R24).
- A part's rectangle was sized as though one pin needed a whole slot,
  which made resistors taller than the gap between rows.

Parts now hang just outside whatever they share a net with, at that
pin's height; nets are routed nearest-first so a net feeding several
parts becomes a chain rather than spokes.  Keep-out is one cell, since
three cells is wider than the row pitch and welded neighbours together.

Co-authored-by: arena-agent <297053741+arena-agent@users.noreply.github.com>
Parts:
- D3, D5, D6, R10, R11, R12, R13, R14, R15, R16, R17, R18, R19, R21, R24, R25, R28, R30, R33: symbol SV16:S0 -> SV16:S1
- FID1, FID2, FID3, FID4, H1, H2, H3, H4, TP1, TP2, TP3, TP4, TP5, TP6: symbol SV16:S1 -> SV16:S2
- J1: symbol SV16:S2 -> SV16:S3
- J10: symbol SV16:S11 -> SV16:S12
- J2: symbol SV16:S3 -> SV16:S4
- J3: symbol SV16:S4 -> SV16:S5
- J4: symbol SV16:S5 -> SV16:S6
- J5: symbol SV16:S6 -> SV16:S7
- J6: symbol SV16:S7 -> SV16:S8
- J7: symbol SV16:S8 -> SV16:S9
- J8: symbol SV16:S9 -> SV16:S10
- J9: symbol SV16:S10 -> SV16:S11
- Q1: symbol SV16:S10 -> SV16:S13
- Q2, Q4: symbol SV16:S10 -> SV16:S14
- SW1, SW2: symbol SV16:S11 -> SV16:S15
- U1: symbol SV16:S12 -> SV16:S16
- U2: symbol SV16:S13 -> SV16:S17
- U3: symbol SV16:S14 -> SV16:S18
- U4: symbol SV16:S15 -> SV16:S19
- U5: symbol SV16:S16 -> SV16:S20
- U6: symbol SV16:S17 -> SV16:S21
- U7: symbol SV16:S18 -> SV16:S22
- U8: symbol SV16:S16 -> SV16:S23
- Y1: symbol SV16:S11 -> SV16:S24
Connections:
- net U3_WP is gone; now on an unnamed net: R17.1
- net TDO: now also J1.10, J2.3
- net TMS: now also J1.9, J2.5
- net led[2]: no longer D4.1, D4.2, R29.2
- net at J6.1: no longer U3.3
- net at J6.2: no longer U3.4
- net PROGRAMN: now reaches Q1.3
- net PROGRAMN: now also J1.3, J1.7, R2.1, SW2.1
- net at J3.12: now also U1.99
- net U2_CLK: now reaches R9.2
- net Y2_XO: now reaches Y2.2
- net Y2_XO: now also C37.1
- net at J4.12: now also U1.135
- net at J2.7: no longer J5.9
- net at J2.8: no longer J5.10
- net A7: now reaches J5.1
- net A6: now reaches J5.2
- net at D5.1: now also R30.2
- net DTR_F: now reaches R25.1
- net DTR_F: now also JP1.2
- net U2_DI: now reaches R10.2
- net at J10.2: now also R24.2
- removed net A2: R10.1, R12.1, R13.2, R14.1, R14.2, R15.1, U2.7, U2.8
- net CC1: no longer names the net of R36.1
- net CCLK: no longer names the net of R9.1
- net CCLK: no longer R8.1
- net CFG_0: no longer names the net of R6.1
- net CFG_1: no longer names the net of R5.1
- net CFG_2: no longer names the net of R7.1
- removed net J10_TX: J10.3, J8.S3, J8.S4, Q1.1, Q1.2, R22.2, R23.2, R24.1, R24.2, R25.2, R26.1, R26.2
- removed net Q4_C: D6.1, D6.2, Q4.1, Q4.2, R31.2, R34.1, R34.2
- net U3_HOLD: no longer names the net of R18.1
- net U3_HOLD: now also U3.4
- net U4_DTR: no longer names the net of JP1.1
- net U4_V3: no longer names the net of C34.1
- net U6_EN: no longer names the net of R41.2
- net U6_EN: no longer C31.1
- net U6_FREQ: no longer names the net of R40.1
- net USB_DP_F: no longer names the net of U8.6
- net ext_rst_n: no longer names the net of C1.1
- net ext_rst_n: no longer R1.1
- net flash_cs_n: no longer names the net of R16.1
- removed net led[0]: D2.1, D2.2, R27.1, R27.2
- removed net led[1]: D3.1, D3.2, R28.1, R28.2
- net led[3]: no longer names the net of R30.1
- net motor_fault_n: no longer names the net of R19.1
- net uart_rx: no longer names the net of R21.2
- net uart_rx: no longer R22.1
- new net: D6.1, R34.1
- new net Q4_B: Q4.1, R31.2
- now unconnected: C38.1, D1.2, D7.2, J3.5, J4.3, L1.2, Q2.1, Q2.2, R32.2, R33.1, R33.2, R44.1, R44.2, U5.6
Other:
- moved on the sheet: C1, C10, C11, C12, C13, C14, C15, C16, C17, C18, C19, C2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

Commit message: Let the router cross wires by their true direction
Two parallel wires side by side looked, to the crossing test, like a
single thick wire running the other way, so legal crossings were
refused and pins ended up sealed behind a band of them.  Each cell now
records which way the copper through it actually runs, and a crossing
is allowed whenever that direction differs from the direction of
travel.

Co-authored-by: arena-agent <297053741+arena-agent@users.noreply.github.com>
Connections:
- net A6: no longer names the net of J5.2
- net A7: no longer names the net of J5.1
- net DTR_F: no longer names the net of R25.1
- net DTR_F: no longer JP1.2
- net U2_CLK: no longer names the net of R9.2
- net clk_25m: no longer names the net of Y1.3
Changed lines of the file:
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@@
     (stroke (width 0) (type default) (color 0 0 0 0))
   )
-  (wire (pts (xy 510.54 393.7) (xy 505.46 393.7) (xy 505.46 347.98) (xy 381 347.98) (xy 381 393.7) (xy 259.08 393.7))
+  (wire (pts (xy 510.54 393.7) (xy 505.46 393.7) (xy 505.46 391.16) (xy 502.92 391.16) (xy 502.92 347.98) (xy 381 347.98) (xy 381 393.7) (xy 259.08 393.7))
     (stroke (width 0) (type default) (color 0 0 0 0))
   )
-  (wire (pts (xy 510.54 383.54) (xy 502.92 383.54) (xy 502.92 345.44) (xy 378.46 345.44) (xy 378.46 375.92) (xy 340.36 375.92) (xy 340.36 383.54) (xy 259.08 383.54))
+  (wire (pts (xy 510.54 383.54) (xy 505.46 383.54) (xy 505.46 345.44) (xy 378.46 345.44) (xy 378.46 375.92) (xy 340.36 375.92) (xy 340.36 383.54) (xy 259.08 383.54))
+    (stroke (width 0) (type default) (color 0 0 0 0))
+  )
+  (wire (pts (xy 510.54 378.46) (xy 500.38 378.46) (xy 500.38 330.2) (xy 457.2 330.2) (xy 457.2 342.9) (xy 375.92 342.9) (xy 375.92 373.38) (xy 337.82 373.38) (xy 337.82 378.46) (xy 259.08 378.46))
+    (stroke (width 0) (type default) (color 0 0 0 0))
+  )
+  (wire (pts (xy 510.54 373.38) (xy 497.84 373.38) (xy 497.84 327.66) (xy 454.66 327.66) (xy 454.66 340.36) (xy 373.38 340.36) (xy 373.38 370.84) (xy 335.28 370.84) (xy 335.28 373.38) (xy 259.08 373.38))
     (stroke (width 0) (type default) (color 0 0 0 0))
   )
@@
     (stroke (width 0) (type default) (color 0 0 0 0))
   )
+  (wire (pts (xy 678.18 398.78) (xy 685.8 398.78) (xy 685.8 388.62) (xy 744.22 388.62) (xy 744.22 213.36) (xy 756.92 213.36) (xy 756.92 198.12) (xy 759.46 198.12) (xy 759.46 195.58) (xy 762 195.58) (xy 762 185.42) (xy 787.4 185.42) (xy 787.4 190.5) (xy 782.32 190.5))
+    (stroke (width 0) (type default) (color 0 0 0 0))
+  )
   (wire (pts (xy 604.52 246.38) (xy 609.6 246.38) (xy 609.6 154.94) (xy 505.46 154.94) (xy 505.46 231.14) (xy 297.18 231.14) (xy 297.18 241.3) (xy 302.26 241.3))
     (stroke (width 0) (type default) (color 0 0 0 0))
@@
     (stroke (width 0) (type default) (color 0 0 0 0))
   )
-  (wire (pts (xy 391.16 388.62) (xy 383.54 388.62) (xy 383.54 406.4) (xy 381 406.4) (xy 381 431.8) (xy 457.2 431.8) (xy 457.2 411.48) (xy 431.8 411.48) (xy 431.8 403.86) (xy 436.88 403.86))
+  (wire (pts (xy 391.16 368.3) (xy 370.84 368.3) (xy 370.84 335.28) (xy 452.12 335.28) (xy 452.12 325.12) (xy 502.92 325.12) (xy 502.92 152.4) (xy 612.14 152.4) (xy 612.14 287.02) (xy 604.52 287.02))
+    (stroke (width 0) (type default) (color 0 0 0 0))
+  )
+  (wire (pts (xy 391.16 388.62) (xy 383.54 388.62) (xy 383.54 406.4) (xy 381 406.4) (xy 381 431.8) (xy 431.8 431.8) (xy 431.8 403.86) (xy 436.88 403.86))
     (stroke (width 0) (type default) (color 0 0 0 0))
   )
@@
     (stroke (width 0) (type default) (color 0 0 0 0))
   )
-  (wire (pts (xy 604.52 1277.62) (xy 609.6 1277.62) (xy 609.6 1247.14) (xy 584.2 1247.14) (xy 584.2 1264.92) (xy 322.58 1264.92) (xy 322.58 1270) (xy 320.04 1270) (xy 320.04 1280.16) (xy 322.58 1280.16) (xy 322.58 1348.74) (xy 327.66 1348.74))
+  (wire (pts (xy 604.52 1277.62) (xy 614.68 1277.62) (xy 614.68 1356.36) (xy 584.2 1356.36) (xy 584.2 1353.82) (xy 322.58 1353.82) (xy 322.58 1348.74) (xy 327.66 1348.74))
     (stroke (width 0) (type default) (color 0 0 0 0))
   )
@@
     (stroke (width 0) (type default) (color 0 0 0 0))
   )
-  (wire (pts (xy 739.14 231.14) (xy 759.46 231.14) (xy 759.46 256.54) (xy 762 256.54) (xy 762 287.02) (xy 789.94 287.02) (xy 789.94 233.68) (xy 787.4 233.68) (xy 787.4 205.74) (xy 782.32 205.74))
+  (wire (pts (xy 739.14 231.14) (xy 749.3 231.14) (xy 749.3 223.52) (xy 746.76 223.52) (xy 746.76 187.96) (xy 759.46 187.96) (xy 759.46 182.88) (xy 789.94 182.88) (xy 789.94 205.74) (xy 782.32 205.74))
+    (stroke (width 0) (type default) (color 0 0 0 0))
+  )
+  (wire (pts (xy 530.86 266.7) (xy 556.26 266.7) (xy 556.26 269.24) (xy 584.2 269.24) (xy 584.2 279.4) (xy 718.82 279.4) (xy 718.82 325.12) (xy 762 325.12) (xy 762 266.7) (xy 769.62 266.7))
     (stroke (width 0) (type default) (color 0 0 0 0))
   )
@@
     (stroke (width 0) (type default) (color 0 0 0 0))
   )
-  (wire (pts (xy 815.34 256.54) (xy 810.26 256.54) (xy 810.26 322.58) (xy 774.7 322.58) (xy 774.7 325.12) (xy 718.82 325.12) (xy 718.82 279.4) (xy 675.64 279.4) (xy 675.64 266.7) (xy 673.1 266.7) (xy 673.1 259.08) (xy 645.16 259.08) (xy 645.16 256.54) (xy 635 256.54))
+  (wire (pts (xy 815.34 256.54) (xy 810.26 256.54) (xy 810.26 322.58) (xy 774.7 322.58) (xy 774.7 327.66) (xy 716.28 327.66) (xy 716.28 281.94) (xy 675.64 281.94) (xy 675.64 266.7) (xy 640.08 266.7) (xy 640.08 256.54) (xy 635 256.54))
     (stroke (width 0) (type default) (color 0 0 0 0))
   )
@@
     (stroke (width 0) (type default) (color 0 0 0 0))
   )
-  (wire (pts (xy 843.28 251.46) (xy 810.26 251.46) (xy 810.26 254) (xy 807.72 254) (xy 807.72 320.04) (xy 772.16 320.04) (xy 772.16 327.66) (xy 716.28 327.66) (xy 716.28 281.94) (xy 673.1 281.94) (xy 673.1 269.24) (xy 670.56 269.24) (xy 670.56 251.46) (xy 662.94 251.46))
+  (wire (pts (xy 843.28 251.46) (xy 838.2 251.46) (xy 838.2 231.14) (xy 822.96 231.14) (xy 822.96 223.52) (xy 820.42 223.52) (xy 820.42 170.18) (xy 718.82 170.18) (xy 718.82 243.84) (xy 675.64 243.84) (xy 675.64 251.46) (xy 662.94 251.46))
     (stroke (width 0) (type default) (color 0 0 0 0))
   )
-  (wire (pts (xy 510.54 251.46) (xy 505.46 251.46) (xy 505.46 264.16) (xy 459.74 264.16) (xy 459.74 261.62) (xy 457.2 261.62) (xy 457.2 254) (xy 431.8 254) (xy 431.8 251.46) (xy 419.1 251.46))
+  (wire (pts (xy 510.54 251.46) (xy 505.46 251.46) (xy 505.46 254) (xy 500.38 254) (xy 500.38 264.16) (xy 459.74 264.16) (xy 459.74 261.62) (xy 457.2 261.62) (xy 457.2 254) (xy 431.8 254) (xy 431.8 251.46) (xy 419.1 251.46))
     (stroke (width 0) (type default) (color 0 0 0 0))
   )
@@
     (stroke (width 0) (type default) (color 0 0 0 0))
   )
-  (wire (pts (xy 510.54 342.9) (xy 505.46 342.9) (xy 505.46 330.2) (xy 457.2 330.2) (xy 457.2 342.9) (xy 259.08 342.9))
+  (wire (pts (xy 510.54 342.9) (xy 505.46 342.9) (xy 505.46 340.36) (xy 502.92 340.36) (xy 502.92 327.66) (xy 500.38 327.66) (xy 500.38 322.58) (xy 449.58 322.58) (xy 449.58 332.74) (xy 368.3 332.74) (xy 368.3 342.9) (xy 259.08 342.9))
     (stroke (width 0) (type default) (color 0 0 0 0))
   )
@@
     (effects (font (size 1.27 1.27)) (justify left))
   )
-  (global_label "A6" (shape input) (at 509.84 379.71 0) (fields_autoplaced)
-    (effects (font (size 1.27 1.27)) (justify left))
-  )
-  (global_label "A6" (shape input) (at 260 379.71 0) (fields_autoplaced)
-    (effects (font (size 1.27 1.27)) (justify left))
-  )
-  (global_label "A7" (shape input) (at 509.84 374.63 0) (fields_autoplaced)
-    (effects (font (size 1.27 1.27)) (justify left))
-  )
-  (global_label "A7" (shape input) (at 260 374.63 0) (fields_autoplaced)
-    (effects (font (size 1.27 1.27)) (justify left))
-  )
-  (global_label "DTR_F" (shape input) (at 678.1 400.03 0) (fields_autoplaced)
-    (effects (font (size 1.27 1.27)) (justify left))
-  )
-  (global_label "DTR_F" (shape input) (at 782.07 191.75 0) (fields_autoplaced)
-    (effects (font (size 1.27 1.27)) (justify left))
-  )
   (symbol (lib_id "SV16:PWR_J9_VIN")
     (at 346.065 1499.9 0)
@@
     (effects (font (size 1.27 1.27)) (justify left))
   )
-  (global_label "U2_CLK" (shape input) (at 391.9 369.55 0) (fields_autoplaced)
-    (effects (font (size 1.27 1.27)) (justify left))
-  )
-  (global_label "U2_CLK" (shape input) (at 604.13 288.27 0) (fields_autoplaced)
-    (effects (font (size 1.27 1.27)) (justify left))
-  )
   (global_label "U2_DI" (shape input) (at 391.9 374.63 0) (fields_autoplaced)
     (effects (font (size 1.27 1.27)) (justify left))
@@
     (effects (font (size 1.27 1.27)) (justify left))
   )
-  (global_label "clk_25m" (shape input) (at 530.16 267.95 0) (fields_autoplaced)
-    (effects (font (size 1.27 1.27)) (justify left))
-  )
-  (global_label "clk_25m" (shape input) (at 770.16 267.95 0) (fields_autoplaced)
-    (effects (font (size 1.27 1.27)) (justify left))
-  )

Commit message: Retry the nets that could not be drawn, with first claim on the sheet
A net's chances depend on when it is routed: the earlier it goes, the
more of the sheet is still empty.  So the generator lays the sheet out,
notes which nets had no path, and runs again with those nets at the
front of the queue.  Three rounds take the unroutable nets from eight
to three.

Co-authored-by: arena-agent <297053741+arena-agent@users.noreply.github.com>
Connections:
- net TCK: now reaches J2.2
- net TCK: now also J1.8
- net INITN: now reaches TP6.1
- net INITN: now also J1.2, R3.1, R31.1
- net Q4_B: no longer names the net of R31.2
- net Q4_B: no longer Q4.1
- net TDO: no longer names the net of J2.3
- net TDO: no longer J1.10
- net TMS: no longer names the net of J2.5
- net TMS: no longer J1.9
- net U2_DI: no longer names the net of R10.2
- net U4_RXD: no longer names the net of R23.1
- net Y2_XO: no longer names the net of Y2.2
- net Y2_XO: no longer C37.1
- net led[2]: no longer names the net of R29.1
