File: hardware/sv16_board/sv16_board.kicad_sch (KiCad schematic)
At the start: 143 parts, among them J1 JTAG, J10 CONSOLE, J2 JTAG-1.27, J3 EXP-A, J4 EXP-B, J5 EXP-C, J6 MOTOR, J7 SPARE (not fitted), J8 USB-C, J9 7-12 V, Q1 2N7002, Q2 BC817, Q4 BC807, SW1 RESET, SW2 RECONFIG, U1 LFE5U-12F-6TG144C, U2 W25Q64JVSSIQ, U3 W25Q64JVSSIQ, U4 CH340G, U5 AP62300TWU-7, U6 MP1584EN, U7 LP5907MFX-2.5, U8 USBLC6-2SC6, Y1 25 MHz ACTIVE XO (4-pin), Y2 12 MHz (CH340G clock)

Commit message: Stand tapping parts clear of the run they tap
Several parts on one net all hung off the same row with their pins on
the near face, which left the wire nowhere to go but straight through
their bodies - PROGRAMN could not reach J1 without crossing Q1, R2 and
J1 itself.  Parts on a net of three or more now sit above or below the
run and tap it with a stub.  Nets of two pins end at the part, so they
stay on the row and keep the straight run.

Co-authored-by: arena-agent <297053741+arena-agent@users.noreply.github.com>
Connections:
- net PROGRAMN: no longer J1.7
- net Y2_XI: now reaches Y2.1
- net Y2_XI: now also C36.1
- net at J4.12: no longer U1.135
- net led[2]_k: now reaches D4.1
- net led[2]_k: now also R29.2
- net at R31.2: now also Q4.1
- net U4_DTR: now reaches JP1.1
- removed net INITN: J1.2, R3.1, R31.1, TP6.1
- net TCK: no longer names the net of J2.2
- net TCK: no longer J1.8
Other:
- moved on the sheet: C1, C34, C36, C37, D1, D2, D3, D4, D5, D6, J10, J8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

Commit message: Slot the parts of one net onto different rows
A single global counter handed whichever part happened to be placed
first the row nearest the run and pushed the rest ever further away, so
SW2 ended up 90 mm from the net it belongs to.  Each net now numbers
its own tapping parts and gives them alternating rows above and below
the run.

247 of the 256 signal pins are now drawn wires; three nets
(PROGRAMN, U2_CLK, led[2]_k - nine pins) still carry labels.

Co-authored-by: arena-agent <297053741+arena-agent@users.noreply.github.com>
Connections:
- net U2_CLK: now reaches R9.2
- net at J4.12: now also U1.135
- net at R31.2: no longer Q4.1
- net at D5.1: no longer R30.2
- net U4_DTR: no longer names the net of JP1.1
- net Y2_XI: no longer names the net of Y2.1
- net Y2_XI: no longer C36.1
Other:
- moved on the sheet: C34, C36, C37, D1, D2, D3, D4, D5, D6, J10, J8, JP1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

Commit message: Never give one FPGA pin to two connectors
Two JTAG headers carry the same four signals, so the FPGA pin for each
of them was being lined up twice - once against each header.  That put
pads 57, 60, 61 and 63 on the FPGA symbol twice, which gave four
duplicate UUIDs and made KiCad refuse the sheet.

An FPGA pin is now claimed by the first connector that wants it; the
second keeps the net and is wired across.  build() also refuses to
emit any symbol that lists a pad twice, so this cannot ship again.

Co-authored-by: arena-agent <297053741+arena-agent@users.noreply.github.com>
Connections:
- net TCK: now reaches J2.6
- net TCK: now also J1.8
- net Q2_C: now reaches D1.1
Other:
- moved on the sheet: J2

Commit message: Rename the LED nets off KiCad's bus notation
led[0]_k and its siblings use square brackets, which KiCad reads as
bus-vector syntax: a label of led[2]_k is not a name it can parse, and
the sheet was rejected on load.  They are now led0_k, led1_k and so on,
renamed at source so the board and the sheet stay in step.

The generator now refuses any net name containing brackets, whitespace
or other characters KiCad reserves.

Co-authored-by: arena-agent <297053741+arena-agent@users.noreply.github.com>
Connections:
- net led[2]_k renamed led2_k
Changed lines of the file:
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@@
     (effects (font (size 1.27 1.27)) (justify left))
   )
-  (global_label "led[2]_k" (shape input) (at 844.13 252.71 0) (fields_autoplaced)
+  (global_label "led2_k" (shape input) (at 844.13 252.71 0) (fields_autoplaced)
     (effects (font (size 1.27 1.27)) (justify left))
   )
-  (global_label "led[2]_k" (shape input) (at 664.13 252.71 0) (fields_autoplaced)
+  (global_label "led2_k" (shape input) (at 664.13 252.71 0) (fields_autoplaced)
     (effects (font (size 1.27 1.27)) (justify left))
   )
